File: hw/sch_pcb/PROGLOG01A.kicad_pcb (KiCad board)
At the start: 2 copper layers, 60.5 x 40.1 mm, 66 parts, among them J1 JUMP_3X2, J10 HEADER_2x01_PARALLEL, J11 HEADER_2x01_PARALLEL, J13 HEADER_2x01_PARALLEL, J14 HEADER_2x01_PARALLEL, J15 HEADER_2x01_PARALLEL, J16 HEADER_2x01_PARALLEL, J17 HEADER_2x01_PARALLEL, J18 HEADER_2x01_PARALLEL, J19 HEADER_2x01_PARALLEL, J2 HEADER_2x01, J20 HEADER_2x01_PARALLEL, J21 HEADER_2x01_PARALLEL, J22 HEADER_2x01_PARALLEL, J23 HEADER_2x01_PARALLEL, J24 HEADER_2x01_PARALLEL, J25 HEADER_2x01_PARALLEL, J26 SATA, J27 HEADER_2x01_PARALLEL, J28 HEADER_2x01_PARALLEL, J29 HEADER_2x01_PARALLEL, J3 HEADER_2x02_PARALLEL, J30 HEADER_2x01_PARALLEL, J31 HEADER_2x01_PARALLEL, J32 HEADER_2x01_PARALLEL, J33 HEADER_2x01_PARALLEL, J34 HEADER_2x01_PARALLEL, J4 HEADER_2x04, J5 HEADER_2x01_PARALLEL, J6 HEADER_2x01_PARALLEL, J7 HEADER_2x01_PARALLEL, J8 HEADER_2x01_PARALLEL, J9 HEADER_2x01_PARALLEL, M1 HOLE, M2 HOLE, M3 HOLE, M4 HOLE, SW1 SW_Push, U1 TPS22919DCK, U2 MIC5504-1.2YM5, U3 AT25SF081-SSHD-X, U4 ICE40UP5K-SG48ITR, X1 ISM92-3351AH24.00

Commit message: Documentation update. Project updated to kicad 6.0.1.
Other:
- net class Default removed
- net class MLAB_power removed
