File: hw/sch_pcb/PROGLOG01B.kicad_sch (KiCad schematic)
At the start: 66 parts, among them J1 JUMP_3X2, J10 HEADER_2x01_PARALLEL, J11 HEADER_2x01_PARALLEL, J13 HEADER_2x01_PARALLEL, J14 HEADER_2x01_PARALLEL, J15 HEADER_2x01_PARALLEL, J16 HEADER_2x01_PARALLEL, J17 HEADER_2x01_PARALLEL, J18 HEADER_2x01_PARALLEL, J19 HEADER_2x01_PARALLEL, J2 HEADER_2x01, J20 HEADER_2x01_PARALLEL, J21 HEADER_2x01_PARALLEL, J22 HEADER_2x01_PARALLEL, J23 HEADER_2x01_PARALLEL, J24 HEADER_2x01_PARALLEL, J25 HEADER_2x01_PARALLEL, J26 SATA, J27 HEADER_2x01_PARALLEL, J28 HEADER_2x01_PARALLEL, J29 HEADER_2x01_PARALLEL, J3 HEADER_2x02_PARALLEL, J30 HEADER_2x01_PARALLEL, J31 HEADER_2x01_PARALLEL, J32 HEADER_2x01_PARALLEL, J33 HEADER_2x01_PARALLEL, J34 HEADER_2x01_PARALLEL, J4 HEADER_2x04, J5 HEADER_2x01_PARALLEL, J6 HEADER_2x01_PARALLEL, J7 HEADER_2x01_PARALLEL, J8 HEADER_2x01_PARALLEL, J9 HEADER_2x01_PARALLEL, M1 HOLE, M2 HOLE, M3 HOLE, M4 HOLE, SW1 SW_Push, U1 TPS22919DCK, U2 MIC5504-1.2YM5, U3 AT25SF081-SSHD-X, U4 ICE40UP5K-SG48ITR, X1 ISM92-3351AH24.00

Commit message: Start a work on updated, fixed version.
Parts:
- U3: value AT25SF081-SSHD-X -> AT25SF081-SSH
Changed lines of the file:
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@@
       (effects (font (size 1.27 1.27)) hide)
     )
-    (property "Datasheet" "http://www.latticesemi.com/Products/FPGAandCPLD/iCE40Ultra" (id 3) (at 181.61 36.83 0)
+    (property "Datasheet" "file:///home/kaklik/Downloads/FPGA-DS-02008-1-9-iCE40-UltraPlus-Family-Data-Sheet.pdf" (id 3) (at 181.61 36.83 0)
       (effects (font (size 1.27 1.27)) hide)
     )
@@
     (pin "42")
     (pin "43")
-  )
-  (symbol (lib_id "PROGLOG01A-rescue:ICE40UP5K-SG48ITR-FPGA_Lattice") (at 217.17 128.27 0) (unit 2)
-    (in_bom yes) (on_board yes)
-    (property "Reference" "U4" (id 0) (at 217.17 155.5496 0))
-    (property "Value" "ICE40UP5K-SG48ITR" (id 1) (at 217.17 157.861 0))
-    (property "Footprint" "Package_DFN_QFN:QFN-48-1EP_7x7mm_P0.5mm_EP5.6x5.6mm" (id 2) (at 217.17 162.56 0)
-      (effects (font (size 1.27 1.27)) hide)
-    )
-    (property "Datasheet" "http://www.latticesemi.com/Products/FPGAandCPLD/iCE40Ultra" (id 3) (at 207.01 102.87 0)
-      (effects (font (size 1.27 1.27)) hide)
-    )
-    (property "UST_ID" "5dc504cb128750448eca1b12" (id 4) (at 217.17 128.27 0)
-      (effects (font (size 1.27 1.27)) hide)
-    )
     (pin "10")
     (pin "11")
@@
     (pin "8")
     (pin "9")
-  )
-  (symbol (lib_id "PROGLOG01A-rescue:ICE40UP5K-SG48ITR-FPGA_Lattice") (at 242.57 137.16 0) (mirror y) (unit 3)
-    (in_bom yes) (on_board yes)
-    (property "Reference" "U4" (id 0) (at 238.76 154.94 0)
-      (effects (font (size 1.27 1.27)) (justify left))
-    )
-    (property "Value" "ICE40UP5K-SG48ITR" (id 1) (at 232.41 151.13 90)
-      (effects (font (size 1.27 1.27)) (justify left))
-    )
-    (property "Footprint" "Package_DFN_QFN:QFN-48-1EP_7x7mm_P0.5mm_EP5.6x5.6mm" (id 2) (at 242.57 171.45 0)
-      (effects (font (size 1.27 1.27)) hide)
-    )
-    (property "Datasheet" "http://www.latticesemi.com/Products/FPGAandCPLD/iCE40Ultra" (id 3) (at 252.73 111.76 0)
-      (effects (font (size 1.27 1.27)) hide)
-    )
-    (property "UST_ID" "5dc504cb128750448eca1b12" (id 4) (at 242.57 137.16 0)
-      (effects (font (size 1.27 1.27)) hide)
-    )
     (pin "1")
     (pin "2")
@@
     (pin "47")
     (pin "48")
+    (pin "24")
+    (pin "29")
+    (pin "30")
+    (pin "49")
+    (pin "5")
+  )
+  (symbol (lib_id "PROGLOG01A-rescue:ICE40UP5K-SG48ITR-FPGA_Lattice") (at 217.17 128.27 0) (unit 2)
+    (in_bom yes) (on_board yes)
+    (property "Reference" "U4" (id 0) (at 217.17 155.5496 0))
+    (property "Value" "ICE40UP5K-SG48ITR" (id 1) (at 217.17 157.861 0))
+    (property "Footprint" "Package_DFN_QFN:QFN-48-1EP_7x7mm_P0.5mm_EP5.6x5.6mm" (id 2) (at 217.17 162.56 0)
+      (effects (font (size 1.27 1.27)) hide)
+    )
+    (property "Datasheet" "file:///home/kaklik/Downloads/FPGA-DS-02008-1-9-iCE40-UltraPlus-Family-Data-Sheet.pdf" (id 3) (at 207.01 102.87 0)
+      (effects (font (size 1.27 1.27)) hide)
+    )
+    (property "UST_ID" "5dc504cb128750448eca1b12" (id 4) (at 217.17 128.27 0)
+      (effects (font (size 1.27 1.27)) hide)
+    )
+    (pin "23")
+    (pin "25")
+    (pin "26")
+    (pin "27")
+    (pin "28")
+    (pin "31")
+    (pin "32")
+    (pin "33")
+    (pin "34")
+    (pin "35")
+    (pin "36")
+    (pin "37")
+    (pin "38")
+    (pin "39")
+    (pin "40")
+    (pin "41")
+    (pin "42")
+    (pin "43")
+    (pin "10")
+    (pin "11")
+    (pin "12")
+    (pin "13")
+    (pin "14")
+    (pin "15")
+    (pin "16")
+    (pin "17")
+    (pin "18")
+    (pin "19")
+    (pin "20")
+    (pin "21")
+    (pin "22")
+    (pin "6")
+    (pin "7")
+    (pin "8")
+    (pin "9")
+    (pin "1")
+    (pin "2")
+    (pin "3")
+    (pin "4")
+    (pin "44")
+    (pin "45")
+    (pin "46")
+    (pin "47")
+    (pin "48")
+    (pin "24")
+    (pin "29")
+    (pin "30")
+    (pin "49")
+    (pin "5")
+  )
+  (symbol (lib_id "PROGLOG01A-rescue:ICE40UP5K-SG48ITR-FPGA_Lattice") (at 242.57 137.16 0) (mirror y) (unit 3)
+    (in_bom yes) (on_board yes)
+    (property "Reference" "U4" (id 0) (at 238.76 154.94 0)
+      (effects (font (size 1.27 1.27)) (justify left))
+    )
+    (property "Value" "ICE40UP5K-SG48ITR" (id 1) (at 232.41 151.13 90)
+      (effects (font (size 1.27 1.27)) (justify left))
+    )
+    (property "Footprint" "Package_DFN_QFN:QFN-48-1EP_7x7mm_P0.5mm_EP5.6x5.6mm" (id 2) (at 242.57 171.45 0)
+      (effects (font (size 1.27 1.27)) hide)
+    )
+    (property "Datasheet" "file:///home/kaklik/Downloads/FPGA-DS-02008-1-9-iCE40-UltraPlus-Family-Data-Sheet.pdf" (id 3) (at 252.73 111.76 0)
+      (effects (font (size 1.27 1.27)) hide)
+    )
+    (property "UST_ID" "5dc504cb128750448eca1b12" (id 4) (at 242.57 137.16 0)
+      (effects (font (size 1.27 1.27)) hide)
+    )
+    (pin "23")
+    (pin "25")
+    (pin "26")
+    (pin "27")
+    (pin "28")
+    (pin "31")
+    (pin "32")
+    (pin "33")
+    (pin "34")
+    (pin "35")
+    (pin "36")
+    (pin "37")
+    (pin "38")
+    (pin "39")
+    (pin "40")
+    (pin "41")
+    (pin "42")
+    (pin "43")
+    (pin "10")
+    (pin "11")
+    (pin "12")
+    (pin "13")
+    (pin "14")
+    (pin "15")
+    (pin "16")
+    (pin "17")
+    (pin "18")
+    (pin "19")
+    (pin "20")
+    (pin "21")
+    (pin "22")
+    (pin "6")
+    (pin "7")
+    (pin "8")
+    (pin "9")
+    (pin "1")
+    (pin "2")
+    (pin "3")
+    (pin "4")
+    (pin "44")
+    (pin "45")
+    (pin "46")
+    (pin "47")
+    (pin "48")
+    (pin "24")
+    (pin "29")
+    (pin "30")
+    (pin "49")
+    (pin "5")
   )
   (symbol (lib_id "PROGLOG01A-rescue:ICE40UP5K-SG48ITR-FPGA_Lattice") (at 115.57 170.18 90) (mirror x) (unit 4)
@@
       (effects (font (size 1.27 1.27)) hide)
     )
-    (property "Datasheet" "http://www.latticesemi.com/Products/FPGAandCPLD/iCE40Ultra" (id 3) (at 90.17 160.02 0)
+    (property "Datasheet" "file:///home/kaklik/Downloads/FPGA-DS-02008-1-9-iCE40-UltraPlus-Family-Data-Sheet.pdf" (id 3) (at 90.17 160.02 0)
       (effects (font (size 1.27 1.27)) hide)
     )
@@
       (effects (font (size 1.27 1.27)) hide)
     )
+    (pin "23")
+    (pin "25")
+    (pin "26")
+    (pin "27")
+    (pin "28")
+    (pin "31")
+    (pin "32")
+    (pin "33")
+    (pin "34")
+    (pin "35")
+    (pin "36")
+    (pin "37")
+    (pin "38")
+    (pin "39")
+    (pin "40")
+    (pin "41")
+    (pin "42")
+    (pin "43")
+    (pin "10")
+    (pin "11")
+    (pin "12")
+    (pin "13")
+    (pin "14")
+    (pin "15")
+    (pin "16")
+    (pin "17")
+    (pin "18")
+    (pin "19")
+    (pin "20")
+    (pin "21")
+    (pin "22")
+    (pin "6")
+    (pin "7")
+    (pin "8")
+    (pin "9")
+    (pin "1")
+    (pin "2")
+    (pin "3")
+    (pin "4")
+    (pin "44")
+    (pin "45")
+    (pin "46")
+    (pin "47")
+    (pin "48")
     (pin "24")
     (pin "29")
@@
       (effects (font (size 1.27 1.27)) (justify left))
     )
-    (property "Value" "AT25SF081-SSHD-X" (id 1) (at 76.2 113.03 0)
+    (property "Value" "AT25SF081-SSH" (id 1) (at 76.2 113.03 0)
       (effects (font (size 1.27 1.27)) (justify left))
     )
@@
       (effects (font (size 1.27 1.27)) hide)
     )
-    (property "Datasheet" "https://www.adestotech.com/wp-content/uploads/DS-AT25SF081_045.pdf" (id 3) (at 73.66 101.6 0)
+    (property "Datasheet" "https://www.renesas.com/us/en/document/dst/at25sf081-datasheet" (id 3) (at 73.66 101.6 0)
       (effects (font (size 1.27 1.27)) hide)
     )
@@
     )
     (path "/00000000-0000-0000-0000-00005e086457"
-      (reference "U3") (unit 1) (value "AT25SF081-SSHD-X") (footprint "Mlab_IO:SOIC-8_3.9x4.9mm_Pitch1.27mm")
+      (reference "U3") (unit 1) (value "AT25SF081-SSH") (footprint "Mlab_IO:SOIC-8_3.9x4.9mm_Pitch1.27mm")
     )
     (path "/00000000-0000-0000-0000-00005d8c3cd5"
